File: _autosave-TPA3255PBTL.kicad_sch (KiCad schematic)
At the start: 46 parts, among them Q2 DMN10H220L, Q3 DMN10H220L, U1 TPA3255DDV

Commit message: Pre mfg, Rev B
Parts:
- removed L6, L7: 10u, Inductor_THT:L_Toroid_Vertical_L22.4mm_W10.2mm_P7.90mm_Vishay_TJ4, symbol Device:L
- added C11, C8: 1u, Capacitor_THT:C_Rect_L7.2mm_W7.2mm_P5.00mm_FKS2_FKP2_MKS2_MKP2, symbol Device:C
- added J6: AC3MAH-AU-PRE, AC3MAH-AU-PRE_AMP, symbol Eli_v6Lib:AC3MAH-AU-PRE
- added TP7, TP8: TestPoint, TestPoint:TestPoint_THTPad_1.0x1.0mm_Drill0.5mm, symbol Connector:TestPoint
- C36, C37: value 12n -> 1u; footprint Capacitor_SMD:C_0805_2012Metric -> Capacitor_THT:C_Rect_L7.2mm_W7.2mm_P5.00mm_FKS2_FKP2_MKS2_MKP2
- L4, L5: value 10u -> 22u
Connections:
- net GND: now also C11.1, J6.1, J6.G, TP7.1, TP8.1; no longer C37.1
- net Load1: now also C8.1, J6.3
- net Load2: now also C37.2, J6.2
- net at C36.1: now also C8.2
- new net: C11.2, C37.1
