File: PowerIn.kicad_sch (KiCad schematic)
At the start: 37 parts, among them J1 Barrel_Jack_Switch, Q1 DMP4015SK3, U2 L78L12_SOT89, U3 L78L33_SO8, U4 NE5532, U5 XL7015

Commit message: Update Layout
Parts:
- C23: footprint Capacitor_SMD:C_1206_3216Metric -> Capacitor_SMD:C_0805_2012Metric
Changed lines of the file:
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@@
       (effects (font (size 1.27 1.27)) (justify left))
     )
-    (property "Footprint" "Capacitor_SMD:C_1206_3216Metric" (id 2) (at 145.7452 107.95 0)
+    (property "Footprint" "Capacitor_SMD:C_0805_2012Metric" (id 2) (at 145.7452 107.95 0)
       (effects (font (size 1.27 1.27)) hide)
     )

Commit message: Update, Post mfg
Parts:
- removed C11: 20u, Capacitor_THT:CP_Radial_D5.0mm_P2.50mm, symbol Device:C_Polarized
- removed C2, C4, C5: C_Polarized, Capacitor_THT:CP_Radial_D12.5mm_P5.00mm, symbol Device:C_Polarized
- removed C8: C, Capacitor_SMD:C_1206_3216Metric, symbol Device:C
- removed D3, D7: LED, LED_THT:LED_D3.0mm_Horizontal_O1.27mm_Z2.0mm, symbol Device:LED
- added C2: 1u, Capacitor_SMD:C_1206_3216Metric, symbol Device:C
- added C4: 100n, Capacitor_SMD:C_0805_2012Metric, symbol Device:C
- added D3, D6: LED_Dual_KAKA, Eli_Lib:IC4_WP934EB_2GD_KNB, symbol Device:LED_Dual_KAKA
- added R34: 470, Resistor_SMD:R_0805_2012Metric, symbol Device:R
- added R35: 2.7k, Resistor_SMD:R_0805_2012Metric, symbol Device:R
- added U6: AD8512, Package_SO:SO-8_3.9x4.9mm_P1.27mm, symbol Amplifier_Operational:NE5532
- C1: value C_Polarized -> 4700u; footprint Capacitor_THT:CP_Radial_D12.5mm_P5.00mm -> Capacitor_THT:CP_Radial_D35.0mm_P10.00mm_SnapIn
- C3, C6, C7: value C -> 1u
- R5: value 1k -> 2.7k
- U4: value NE5532 -> AD8512
Connections:
- net +12V: now also R5.2, C4.1, U6.8 (V+)
- net +15V: now also D3.4 (K2)
- net +3V3: now also R34.1
- net +48V: now also C2.1, D3.2 (K1)
- net GND: now also C2.2, C4.2, D6.1 (A1), D6.3 (A2), R35.2, U6.4 (V-); no longer R5.2
- net at R5.1: now also D6.2 (K1)
- net at R3.1: now also D3.1 (A1)
- new net: D3.3 (A2), R35.1
- new net: D6.4 (K2), R34.2
Other:
- note added: "GRM31CR72A105KA01L Under heat sink"
- note added: "SLPX472M080H3P3"
- moved on the sheet: R3

Commit message: Pre mfg, Rev B
Parts:
- C28, C30, C9: footprint Capacitor_THT:CP_Radial_D5.0mm_P2.50mm -> Capacitor_THT:CP_Radial_D6.3mm_P2.50mm
- U5: footprint Package_TO_SOT_SMD:TO-252-5_TabPin6 -> Eli_Lib:XL7015E1
