File: SignalIn.kicad_sch (KiCad schematic)
At the start: 21 parts, among them J2 Conn_Coaxial, J3 Conn_02x04_Odd_Even, U4 NE5532

Commit message: Update, Post mfg
Parts:
- removed C17: 10n, Capacitor_SMD:C_0805_2012Metric, symbol Device:C
- removed C18: 1n, Capacitor_SMD:C_0805_2012Metric, symbol Device:C
- removed C19: 100p, Capacitor_SMD:C_0805_2012Metric, symbol Device:C
- removed C20, C27: 100n, Capacitor_SMD:C_0805_2012Metric, symbol Device:C
- removed J2: Conn_Coaxial, Connector_Coaxial:BNC_TEConnectivity_1478035_Horizontal, symbol Connector:Conn_Coaxial
- removed J3: Conn_02x04_Odd_Even, Connector_PinHeader_2.54mm:PinHeader_2x04_P2.54mm_Vertical, symbol Connector_Generic:Conn_02x04_Odd_Even
- removed R10, R8: 10k, Resistor_SMD:R_0805_2012Metric, symbol Device:R
- added C43: 10n, Capacitor_SMD:C_0805_2012Metric, symbol Device:C
- added C44, C45: 330p, Capacitor_SMD:C_0805_2012Metric, symbol Device:C
- added C5, C8: 100n, Capacitor_SMD:C_0805_2012Metric, symbol Device:C
- added J2: AC3FAH2-XLR, Eli_Lib:AC3FAH2-F-XLR, symbol Eli_v6Lib:AC3FAH2-XLR
- added R31, R37, R38, R40, R42, R43, R44, R45, R46: 10k, Resistor_SMD:R_0805_2012Metric, symbol Device:R
- added R36, R39: 1k, Resistor_SMD:R_0805_2012Metric, symbol Device:R
- added R41: DNP, Resistor_SMD:R_0805_2012Metric, symbol Device:R
- added S1: PB400EEQX, Eli_Lib:SW_PB400EEQX, symbol Eli_v6Lib:PB400EEQX
- added TP2, TP3, TP4, TP6, TP7: TestPoint, TestPoint:TestPoint_THTPad_1.0x1.0mm_Drill0.5mm, symbol Connector:TestPoint
- added U6, U7: AD8512, Package_SO:SO-8_3.9x4.9mm_P1.27mm, symbol Amplifier_Operational:NE5532
- C16: value 100n -> 10n
- C21, C22: value 1u -> 47u; footprint Capacitor_SMD:C_0805_2012Metric -> Capacitor_SMD:C_1206_3216Metric_Pad1.33x1.80mm_HandSolder
- R20: value 10k -> 4.7k
- U4: value NE5532 -> AD8512
Connections:
- net +12V: now also C5.2, U7.8 (V+)
- net FiltInA: now also TP3.1
- net FiltInB: now also TP4.1
- net GND: now also C5.1, C8.1, J2.1, J2.G, R36.2, R39.1; no longer R11.2
- net Input: now also J2.3, S1.1
- net at R11.1: now also C43.2, S1.4; no longer U4.5 (+)
- net at C26.2, R20.1, R9.2: now also U6.3 (+); no longer U4.3 (+)
- net at C21.1, R12.1, R22.2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: now also C45.2
- net at R21.2, R22.1, U4.2 (-): now also C45.1
- net at C16.2: now also R21.1, S1.2
- new net: C44.1, R11.2, R31.1, U4.3 (+)
- new net: R36.1, R37.2, U7.5 (+)
- new net: R43.1, R45.2, U6.5 (+)
- new net: C8.2, TP7.1, U7.4 (V-)
- new net: R38.1, R39.2, U7.3 (+)
- new net: R42.1, R44.2, U7.1
- new net: R41.1, R42.2, U7.2 (-)
- new net: R40.1, R41.2, U7.6 (-)
- new net: R40.2, R43.2, U7.7
- new net: R44.1, R46.2, U6.6 (-)
- new net: C43.1, J2.2, S1.3
- new net: R46.1, TP6.1, U6.7
- new net +3V8: C44.2, R31.2, R45.1, TP2.1, U4.5 (+), U6.1, U6.2 (-)
- new net Load1: R37.1
- new net Load2: R38.2
Other:
- moved on the sheet: C16, C21, C22, C26, R12, R13, R20, R21, R22, R9, U4A, U4B

Commit message: Pre mfg, Rev B
Parts:
- removed C8: 100n, Capacitor_SMD:C_0805_2012Metric, symbol Device:C
- removed TP7: TestPoint, TestPoint:TestPoint_THTPad_1.0x1.0mm_Drill0.5mm, symbol Connector:TestPoint
- added H1, H2, H3: MountingHole_Pad, MountingHole:MountingHole_3.2mm_M3_Pad_Via, symbol Mechanical:MountingHole_Pad
- added J3: Screw_Terminal_01x02, TerminalBlock_Phoenix:TerminalBlock_Phoenix_MKDS-1,5-2-5.08_1x02_P5.08mm_Horizontal, symbol Connector:Screw_Terminal_01x02
- added J4, J5: Conn_01x02_Pin, Connector_PinHeader_1.27mm:PinHeader_1x02_P1.27mm_Vertical, symbol Connector:Conn_01x02_Pin
- added R47, R48, R49: 10k, Resistor_SMD:R_0805_2012Metric, symbol Device:R
- added R50, R51: 1k, Resistor_SMD:R_0805_2012Metric, symbol Device:R
- added RV1: 500, Potentiometer_THT:Potentiometer_Bourns_3296W_Vertical, symbol Device:R_Potentiometer_Trim
- R22: value 10k -> 4.7k
Connections:
- net +3V8: now also R48.2
- net FiltInA: now also R51.2
- net FiltInB: now also R50.2
- net GND: now also U7.4 (V-), H1.1, H2.1, H3.1
- net Load1: now also J3.1 (Pin_1)
- net Load2: now also J3.2 (Pin_2)
- net at C44.1, R11.2, R31.1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: now also R47.2, R48.1
- net at C22.1, R13.2, U4.7: now also J4.1 (Pin_1)
- net at C45.1, R21.2, R22.1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: now also R49.2
- net at C21.1, C45.2, R12.1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: now also J5.1 (Pin_1), RV1.2, RV1.3; no longer R22.2
- net at C16.2, R21.1, S1.2: now also R49.1
- net at C43.2, R11.1, S1.4: now also R47.1
- new net: R22.2, RV1.1
- new net: J4.2 (Pin_2), R50.1
- new net: J5.2 (Pin_2), R51.1
Other:
- moved on the sheet: C16, C21, C22, C43, C44, C45, J2, R11, R12, R13, R21, R22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

Commit message: Add testing/ update README/ Current control
Parts:
- added J7: AC3FAH2-XLR, Eli_Lib:AC3FAH2-F-XLR, symbol Eli_v6Lib:AC3FAH2-XLR
- C21, C22: value 47u -> 22u
Connections:
- net GND: now also J7.1, J7.G
- net Input: now also J7.3
- net Load1: now also J3.2 (Pin_2); no longer J3.1 (Pin_1)
- net Load2: now also J3.1 (Pin_1); no longer J3.2 (Pin_2)
- net at C43.1, J2.2, S1.3: now also J7.2
