File: TPA3255PBTL.kicad_pcb (KiCad board)
At the start: 4 copper layers, 116 x 72 mm, 89 parts, among them J1 Barrel_Jack_Switch, J2 Conn_Coaxial, J3 Conn_02x04_Odd_Even, Q1 DMP4015SK3, Q2 DMN10H220L, Q3 DMN10H220L, SW1 SW_Push_Dual, U1 TPA3255DDV, U2 L78L12_SOT89, U3 L78L33_SO8, U4 NE5532, U5 XL7015

Commit message: Update Layout
Parts:
- removed C14: 100n, Capacitor_SMD:C_1206_3216Metric
- added C40: 1u, Capacitor_SMD:C_0805_2012Metric, F.Cu at (120.8, 89.2)
- added C41: 1u, Capacitor_SMD:C_0805_2012Metric, F.Cu at (125.0, 84.2)
- added C42: 100n, Capacitor_SMD:C_0805_2012Metric, B.Cu at (116.5, 84.5)
- added R29: 22k, Resistor_SMD:R_0805_2012Metric, F.Cu at (110.8, 86.5)
- added R30: 30k, Resistor_SMD:R_0805_2012Metric, F.Cu at (110.8, 89.8)
- C13, C23, C32, C33, C34, C35: footprint Capacitor_SMD:C_1206_3216Metric -> Capacitor_SMD:C_0805_2012Metric
- C24, C25: footprint Capacitor_SMD:C_1206_3216Metric -> Capacitor_SMD:C_0805_2012Metric; moved to B.Cu
- C6, C7, U1: moved to B.Cu
- moved C6 52.2 mm to (133.8, 88.5)
- moved C36 49.7 mm to (147.2, 56.0)
- moved C3 48.4 mm to (134.5, 82.5)
- moved C8 46.9 mm to (124.2, 87.2), turned to 180 degrees
- moved C37 46.5 mm to (140.8, 103.5)
- moved C7 45.7 mm to (134.5, 82.5)
- moved C25 20.1 mm to (123.2, 95.7), turned to -90 degrees
- moved C24 19.2 mm to (122.7, 77.0), turned to 180 degrees
- moved C32 18.4 mm to (130.0, 94.5), turned to 180 degrees
- moved C35 17.8 mm to (130.0, 74.5), turned to 180 degrees
- moved R6 17.1 mm to (122.4, 77.2)
- moved R7 16.9 mm to (123.1, 94.2)
- moved C33 16.6 mm to (130.0, 97.0), turned to 180 degrees
- moved C34 16.1 mm to (130.0, 77.0), turned to 180 degrees
- moved C13 13.9 mm to (118.5, 80.0)
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Connections:
- net Net-(C36-Pad1) renamed Load1
- net Net-(C37-Pad2) renamed Load2
- net Net-(D1-Pad2) renamed Power_IN
- U1 pad 14: unconnected-(U1-Pad14) -> AVDD
Routing:
- net +12V: track 0.00 -> 61.6 mm, vias 0 -> 6
- net GND: track 0.00 -> 55.4 mm, vias 0 -> 32
- net CLIP_OTW: track 0.00 -> 54.0 mm, vias 0 -> 3
- net +48V: track 0.00 -> 53.3 mm, vias 0 -> 12
- net Fault: track 0.00 -> 43.1 mm, vias 0 -> 1
- net RST_: track 0.00 -> 34.2 mm, vias 0 -> 1
- net +15V: track 0.00 -> 33.4 mm
- net OUTB: track 0.00 -> 31.2 mm, vias 0 -> 7
- net +3V3: track 0.00 -> 22.4 mm
- net Input: track 0.00 -> 21.3 mm
- net OUTC: track 0.00 -> 20.9 mm, vias 0 -> 2
- net Net-(C21-Pad1): track 0.00 -> 17.5 mm
- net Net-(D6-Pad2): track 0.00 -> 16.7 mm
- net Net-(R10-Pad2): track 0.00 -> 16.2 mm, vias 0 -> 2
- net FiltInB: track 0.00 -> 15.5 mm, vias 0 -> 1
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- added copper zone on In2.Cu, net +12V
- added copper zone on In2.Cu, net +48V
- added copper zone on In1.Cu, net GND
- added copper zone on F.Cu, net Load1
- added copper zone on F.Cu, net Load2
- added copper zone on F.Cu, net OUTB
- added copper zone on B.Cu, net OUTC
- added copper zone on F.Cu, net Power_IN

Commit message: Update, Post mfg
Parts:
- removed C11: 20u, Capacitor_THT:CP_Radial_D5.0mm_P2.50mm
- removed C39: 4.7n, Capacitor_THT:C_Rect_L18.0mm_W6.0mm_P15.00mm_FKS3_FKP3
- removed D7: LED, LED_THT:LED_D3.0mm_Horizontal_O1.27mm_Z2.0mm
- removed J3: Conn_02x04_Odd_Even, Connector_PinHeader_2.54mm:PinHeader_2x04_P2.54mm_Vertical
- removed SW1: SW_Push_Dual, Button_Switch_SMD:SW_SPST_Omron_B3FS-105xP
- added C14: 1u, Capacitor_THT:C_Rect_L7.2mm_W7.2mm_P5.00mm_FKS2_FKP2_MKS2_MKP2, F.Cu at (168.9, 88.6)
- added C43: 10n, Capacitor_SMD:C_0805_2012Metric, F.Cu at (91.0, 102.0)
- added C44: 330p, Capacitor_SMD:C_0805_2012Metric, F.Cu at (103.5, 115.2)
- added C45: 330p, Capacitor_SMD:C_0805_2012Metric, F.Cu at (105.6, 118.8)
- added L4: 10u, Inductor_THT:L_Toroid_Vertical_L22.4mm_W10.2mm_P7.90mm_Vishay_TJ4, F.Cu at (188.5, 91.0)
- added L5: 10u, Inductor_THT:L_Toroid_Vertical_L22.4mm_W10.2mm_P7.90mm_Vishay_TJ4, F.Cu at (188.5, 96.8)
- added L6: 10u, Inductor_THT:L_Toroid_Vertical_L22.4mm_W10.2mm_P7.90mm_Vishay_TJ4, F.Cu at (198.0, 66.0)
- added L7: 10u, Inductor_THT:L_Toroid_Vertical_L22.4mm_W10.2mm_P7.90mm_Vishay_TJ4, F.Cu at (190.3, 118.5)
- added Q4: DMN10H220L, Package_TO_SOT_SMD:SOT-23, F.Cu at (101.5, 91.0)
- added Q5: DMN10H220L, Package_TO_SOT_SMD:SOT-23, F.Cu at (97.0, 91.0)
- added R31: 10k, Resistor_SMD:R_0805_2012Metric, F.Cu at (105.7, 115.2)
- added R32: 47k, Resistor_SMD:R_0805_2012Metric, F.Cu at (101.4, 93.9)
- added R33: 47k, Resistor_SMD:R_0805_2012Metric, F.Cu at (96.9, 93.9)
- added R34: 470, Resistor_SMD:R_0805_2012Metric, F.Cu at (82.8, 71.6)
- added R35: 2.7k, Resistor_SMD:R_0805_2012Metric, F.Cu at (82.9, 66.3)
- added R36: 1k, Resistor_SMD:R_0805_2012Metric, F.Cu at (123.5, 126.2)
- added R37: 10k, Resistor_SMD:R_0805_2012Metric, F.Cu at (120.0, 126.2)
- added R38: 10k, Resistor_SMD:R_0805_2012Metric, F.Cu at (120.0, 128.8)
- added R39: 1k, Resistor_SMD:R_0805_2012Metric, F.Cu at (123.5, 128.8)
- added R40: 10k, Resistor_SMD:R_0805_2012Metric, F.Cu at (115.2, 127.8)
- added R41: DNP, Resistor_SMD:R_0805_2012Metric, F.Cu at (110.3, 124.1)
- added R42: 10k, Resistor_SMD:R_0805_2012Metric, F.Cu at (105.2, 126.8)
- added R43: 10k, Resistor_SMD:R_0805_2012Metric, F.Cu at (101.5, 102.5)
- added R44: 10k, Resistor_SMD:R_0805_2012Metric, F.Cu at (99.0, 102.5)
- added R45: 10k, Resistor_SMD:R_0805_2012Metric, F.Cu at (101.2, 99.0)
- added R46: 10k, Resistor_SMD:R_0805_2012Metric, F.Cu at (99.0, 99.0)
- added S1: PB400EEQX, Eli_Lib:SW_PB400EEQX, F.Cu at (87.7, 96.1)
- added S2: PB400OAQX, Eli_Lib:SW_PB400EEQX, F.Cu at (87.7, 77.3)
- added TP1: TestPoint, TestPoint:TestPoint_THTPad_1.0x1.0mm_Drill0.5mm, F.Cu at (92.0, 79.4)
- added TP2: TestPoint, TestPoint:TestPoint_THTPad_1.0x1.0mm_Drill0.5mm, F.Cu at (107.6, 112.2)
- added TP3: TestPoint, TestPoint:TestPoint_THTPad_1.0x1.0mm_Drill0.5mm, F.Cu at (104.5, 101.0)
- added TP4: TestPoint, TestPoint:TestPoint_THTPad_1.0x1.0mm_Drill0.5mm, F.Cu at (107.0, 101.0)
- added TP5: TestPoint, TestPoint:TestPoint_THTPad_1.0x1.0mm_Drill0.5mm, F.Cu at (92.1, 82.9)
- added TP6: TestPoint, TestPoint:TestPoint_THTPad_1.0x1.0mm_Drill0.5mm, F.Cu at (95.2, 98.0)
- added TP7: TestPoint, TestPoint:TestPoint_THTPad_1.0x1.0mm_Drill0.5mm, F.Cu at (105.2, 129.8)
- added U6: AD8512, Package_SO:SO-8_3.9x4.9mm_P1.27mm, F.Cu at (99.6, 108.0)
- added U7: AD8512, Package_SO:SO-8_3.9x4.9mm_P1.27mm, F.Cu at (110.2, 127.8)
- C1: value C_Polarized -> 4700u; footprint Capacitor_THT:CP_Radial_D12.5mm_P5.00mm -> Capacitor_THT:CP_Radial_D35.0mm_P10.00mm_SnapIn
- C16, C20, C27: value 100n -> 10n
- C17: value 10n -> 1u; footprint Capacitor_SMD:C_0805_2012Metric -> Capacitor_THT:C_Rect_L7.2mm_W7.2mm_P5.00mm_FKS2_FKP2_MKS2_MKP2
- C19: value 100p -> 1n
- C2: value C_Polarized -> 1u; footprint Capacitor_THT:CP_Radial_D12.5mm_P5.00mm -> Capacitor_SMD:C_1206_3216Metric
- C21, C22: value 1u -> 47u; footprint Capacitor_SMD:C_0805_2012Metric -> Capacitor_SMD:C_1206_3216Metric_Pad1.33x1.80mm_HandSolder
- C24, C25, U1: moved to F.Cu
- C3: value C -> 1u
- C36, C37: value 220n -> 12n; footprint Capacitor_THT:C_Rect_L33.0mm_W20.0mm_P27.50mm_MKS4 -> Capacitor_SMD:C_0805_2012Metric
- C38: value 4.7n -> 47u; footprint Capacitor_THT:C_Rect_L18.0mm_W6.0mm_P15.00mm_FKS3_FKP3 -> Capacitor_SMD:C_1206_3216Metric_Pad1.33x1.80mm_HandSolder
- C4, C5: value C_Polarized -> 100n; footprint Capacitor_THT:CP_Radial_D12.5mm_P5.00mm -> Capacitor_SMD:C_0805_2012Metric
- C42: value 100n -> 47n; moved to F.Cu
- C6, C7: value C -> 1u; moved to F.Cu
- C8: value C -> 100n; footprint Capacitor_SMD:C_1206_3216Metric -> Capacitor_SMD:C_0805_2012Metric
- D3, D5, D6: value LED -> LED_Dual_KAKA; footprint LED_THT:LED_D3.0mm_Horizontal_O1.27mm_Z2.0mm -> Eli_Lib:IC4_WP934EB_2GD_KNB
- J2: value Conn_Coaxial -> AC3FAH2-XLR; footprint Connector_Coaxial:BNC_TEConnectivity_1478035_Horizontal -> Eli_Lib:AC3FAH2-F-XLR
- R10, R8: value 10k -> 3R3
- R20: value 10k -> 4.7k
- R5: value 1k -> 2.7k
- U4: value NE5532 -> AD8512
- moved C17 89.3 mm to (182.0, 109.5), turned to -90 degrees
- moved C38 76.7 mm to (104.9, 92.1), turned to -90 degrees
- moved C5 72.1 mm to (113.2, 123.3), turned to -90 degrees
- moved C18 70.1 mm to (162.1, 92.8), turned to 180 degrees
- moved C19 70.1 mm to (162.0, 120.5)
- moved C37 63.9 mm to (203.0, 118.0), turned to -90 degrees
- moved C20 63.7 mm to (165.2, 88.8), turned to 180 degrees
- moved R8 61.6 mm to (161.7, 88.8), turned to 0 degrees
- moved C1 58.2 mm to (161.6, 62.4)
- moved C36 56.6 mm to (202.2, 69.5), turned to -90 degrees
- moved C4 48.4 mm to (95.8, 102.5), turned to 90 degrees
- moved C8 47.9 mm to (102.2, 129.8), turned to 0 degrees
- moved C27 41.7 mm to (162.0, 123.0), turned to 0 degrees
- moved R10 40.0 mm to (158.5, 123.0), turned to 180 degrees
- moved C2 33.9 mm to (137.0, 83.3), turned to -90 degrees
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Connections:
- net OUTC renamed OUTA
- C17 pad 1: Input -> GND
- C17 pad 2: Net-(C17-Pad2) -> OUTB2
- C18 pad 1: Input -> OUTA2
- C18 pad 2: Net-(C18-Pad2) -> GND
- C19 pad 1: Input -> GND
- C19 pad 2: Net-(C19-Pad2) -> OUTB2
- C20 pad 1: Net-(C20-Pad1) -> OUTA2
- C26 pad 2: Net-(U4-Pad3) -> Net-(C26-Pad2)
- C27 pad 1: GND -> Net-(C27-Pad1)
- C27 pad 2: Net-(R10-Pad2) -> OUTB2
- C36 pad 1: Load1 -> Net-(C36-Pad1)
- C37 pad 2: Load2 -> Net-(C37-Pad2)
- C38 pad 1: Load1 -> GND
- C38 pad 2: GND -> Net-(C38-Pad2)
- C4 pad 1: +48V -> +12V
- C5 pad 1: +48V -> GND
- C5 pad 2: GND -> +12V
- C8 pad 1: +48V -> GND
- C8 pad 2: GND -> Net-(U7-Pad4)
- J2 pad 1: Input -> GND
- J2 pad 2: GND -> Net-(C43-Pad1)
- L2 pad 2: Load1 -> OUTA2
- L3 pad 2: Load2 -> OUTB2
- Q2 pad 3: Net-(D5-Pad2) -> Net-(D5-Pad4)
- Q3 pad 3: Net-(D6-Pad2) -> Net-(D5-Pad2)
- R10 pad 1: +12V -> Net-(C27-Pad1)
- R10 pad 2: Net-(R10-Pad2) -> GND
- R11 pad 1: Net-(R10-Pad2) -> Net-(C43-Pad2)
- R11 pad 2: GND -> Net-(C44-Pad1)
- R20 pad 1: Net-(U4-Pad3) -> Net-(C26-Pad2)
- R21 pad 1: Net-(C20-Pad2) -> Net-(C16-Pad2)
- R25 pad 1: Net-(D5-Pad2) -> Net-(D5-Pad4)
- R28 pad 1: Net-(D6-Pad2) -> Net-(D5-Pad2)
- R5 pad 1: Net-(D7-Pad1) -> Net-(D6-Pad2)
- R5 pad 2: GND -> +12V
- R8 pad 1: Net-(C20-Pad1) -> GND
- R8 pad 2: GND -> Net-(C20-Pad2)
- R9 pad 2: Net-(U4-Pad3) -> Net-(C26-Pad2)
- U4 pad 3: Net-(U4-Pad3) -> Net-(C44-Pad1)
- U4 pad 5: Net-(R10-Pad2) -> +3V8
Routing:
- net Load1: track 0.00 -> 105.4 mm, vias 0 -> 1
- net Load2: track 0.00 -> 77.6 mm, vias 0 -> 1
- net Net-(R42-Pad1): track 0.00 -> 42.8 mm, vias 0 -> 2
- net Net-(R40-Pad2): track 0.00 -> 39.6 mm, vias 0 -> 2
- net +3V8: track 0.00 -> 36.3 mm, vias 0 -> 2
- net Net-(C45-Pad1): track 7.82 -> 39.4 mm, vias 0 -> 2
- net +15V: track 33.4 -> 7.40 mm, vias 0 -> 5
- net +3V3: track 22.4 -> 47.6 mm, vias 0 -> 3
- net FiltInA: track 15.3 -> 40.5 mm, vias 1 -> 0
- net Net-(C26-Pad2): track 0.00 -> 24.4 mm, vias 0 -> 2
- net FiltInB: track 15.5 -> 38.9 mm, vias 1 -> 0
- net Net-(C44-Pad1): track 0.00 -> 23.0 mm, vias 0 -> 3
- net RST_: track 34.2 -> 52.1 mm, vias 1 -> 2
- net Net-(R38-Pad1): track 0.00 -> 16.9 mm
- net Net-(C43-Pad2): track 0.00 -> 16.8 mm
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- added copper zone on In2.Cu, net +15V
- added copper zone on F.Cu, net +48V
- added copper zone on F.Cu, net OUTA
- added copper zone on F.Cu, net OUTA2
- added copper zone on B.Cu, net OUTB
- added copper zone on F.Cu, net OUTB2
Other:
- board size 116 x 72 mm -> 136.6 x 87.2 mm
- board text added: "+3.8V"
- board text added: "Fault"
- board text added: "Filt Sig.+/-"
- board text added: "Vmon"
- board text added: "Vmon VS-"
- board text added: "_RST"

Commit message: Pre mfg, Rev B
Parts:
- removed L6, L7: 10u, Inductor_THT:L_Toroid_Vertical_L22.4mm_W10.2mm_P7.90mm_Vishay_TJ4
- added C11: 1u, Capacitor_THT:C_Rect_L7.2mm_W7.2mm_P5.00mm_FKS2_FKP2_MKS2_MKP2, F.Cu at (190.5, 112.0)
- added H1: MountingHole_Pad, MountingHole:MountingHole_3.2mm_M3_Pad_Via, F.Cu at (151.0, 127.4)
- added H2: MountingHole_Pad, MountingHole:MountingHole_3.2mm_M3_Pad_Via, F.Cu at (151.0, 48.0)
- added H3: MountingHole_Pad, MountingHole:MountingHole_3.2mm_M3_Pad_Via, F.Cu at (206.0, 127.0)
- added J3: Screw_Terminal_01x02, TerminalBlock_Phoenix:TerminalBlock_Phoenix_MKDS-1,5-2-5.08_1x02_P5.08mm_Horizontal, F.Cu at (205.5, 90.5)
- added J4: Conn_01x02_Pin, Connector_PinHeader_1.27mm:PinHeader_1x02_P1.27mm_Vertical, F.Cu at (108.2, 109.5)
- added J5: Conn_01x02_Pin, Connector_PinHeader_1.27mm:PinHeader_1x02_P1.27mm_Vertical, F.Cu at (104.8, 109.4)
- added J6: AC3MAH-AU-PRE, Eli_Lib:AC3MAH-AU-PRE_AMP, F.Cu at (192.2, 61.0)
- added R47: 10k, Resistor_SMD:R_0805_2012Metric, F.Cu at (93.4, 110.6)
- added R48: 10k, Resistor_SMD:R_0805_2012Metric, F.Cu at (107.8, 115.2)
- added R49: 10k, Resistor_SMD:R_0805_2012Metric, F.Cu at (91.2, 100.6)
- added R50: 1k, Resistor_SMD:R_0805_2012Metric, F.Cu at (107.4, 105.0)
- added R51: 1k, Resistor_SMD:R_0805_2012Metric, F.Cu at (105.2, 105.0)
- added R52: 10k, Resistor_SMD:R_0805_2012Metric, F.Cu at (96.2, 85.9)
- added RV1: 500, Potentiometer_THT:Potentiometer_Bourns_3296W_Vertical, F.Cu at (95.0, 128.1)
- added TP8: TestPoint, TestPoint:TestPoint_THTPad_1.0x1.0mm_Drill0.5mm, F.Cu at (95.2, 96.0)
- C28, C30, C9: footprint Capacitor_THT:CP_Radial_D5.0mm_P2.50mm -> Capacitor_THT:CP_Radial_D6.3mm_P2.50mm
- C36, C37: value 12n -> 1u; footprint Capacitor_SMD:C_0805_2012Metric -> Capacitor_THT:C_Rect_L7.2mm_W7.2mm_P5.00mm_FKS2_FKP2_MKS2_MKP2
- C8: value 100n -> 1u; footprint Capacitor_SMD:C_0805_2012Metric -> Capacitor_THT:C_Rect_L7.2mm_W7.2mm_P5.00mm_FKS2_FKP2_MKS2_MKP2
- L4, L5: value 10u -> 22u
- R22: value 10k -> 4.7k
- U5: footprint Package_TO_SOT_SMD:TO-252-5_TabPin6 -> Eli_Lib:XL7015E1
- moved C8 107.1 mm to (194.9, 76.0)
- moved TP7 90.7 mm to (73.0, 45.0)
- moved C21 7.46 mm to (104.8, 100.2)
- moved C22 7.46 mm to (107.8, 100.2)
- moved C37 7.38 mm to (198.7, 112.0), turned to 0 degrees
- moved C36 6.56 mm to (203.1, 76.0), turned to 0 degrees
- moved TP4 4.60 mm to (106.8, 96.4)
- moved TP3 4.60 mm to (104.6, 96.4)
- moved R7 4.49 mm to (128.0, 76.5)
- moved R6 4.23 mm to (127.5, 95.0)
- moved R36 3.64 mm to (120.0, 125.2), turned to 180 degrees
- moved R37 3.64 mm to (123.5, 125.2), turned to 180 degrees
- moved R38 3.50 mm to (123.5, 128.8), turned to 0 degrees
- moved R39 3.50 mm to (120.0, 128.8), turned to 0 degrees
- moved C28 3.40 mm to (106.5, 74.5)
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Connections:
- C21 pad 1: Net-(C21-Pad1) -> Net-(J5-Pin_1)
- C37 pad 1: GND -> Net-(C11-Pad2)
- C37 pad 2: Net-(C37-Pad2) -> Load2
- C45 pad 2: Net-(C21-Pad1) -> Net-(J5-Pin_1)
- C8 pad 1: GND -> Load1
- C8 pad 2: Net-(U7-Pad4) -> Net-(C36-Pad1)
- R12 pad 1: Net-(C21-Pad1) -> Net-(J5-Pin_1)
- R22 pad 2: Net-(C21-Pad1) -> Net-(R22-Pad2)
- TP7 pad 1: Net-(U7-Pad4) -> GND
- U4 pad 1: Net-(C21-Pad1) -> Net-(J5-Pin_1)
- U7 pad 4: Net-(U7-Pad4) -> GND
Routing:
- net Load2: track 77.6 -> 136.7 mm
- net Net-(J5-Pin_1): track 0.00 -> 44.4 mm, vias 0 -> 1
- net Net-(C21-Pad1): track 31.8 -> 0.00 mm
- net Load1: track 105.4 -> 131.2 mm
- net Net-(J4-Pin_1): track 12.3 -> 20.8 mm
- net Net-(R22-Pad2): track 0.00 -> 6.20 mm
- net +3V3: track 47.6 -> 53.2 mm
- net +48V: track 52.7 -> 47.1 mm
- net Net-(C37-Pad2): track 4.99 -> 0.00 mm
- net +12V: track 67.8 -> 63.0 mm, vias 13 -> 15
- net Net-(U7-Pad4): track 4.49 -> 0.00 mm
- net Net-(U4A-+): track 23.0 -> 26.6 mm
- net Net-(C43-Pad2): track 16.8 -> 20.1 mm
- net Net-(C11-Pad2): track 0.00 -> 3.20 mm
- net GVDD_AB: track 7.30 -> 4.28 mm
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Other:
- board size 136.6 x 87.2 mm -> 138 x 87.2 mm
- board text added: "GND"
- board text removed: "Vmon VS-"

Commit message: Add testing/ update README/ Current control
Parts:
- added J7: AC3FAH2-XLR, Eli_Lib:AC3FAH2-F-XLR, F.Cu at (199.2, 124.5)
- moved H3 22.0 mm to (184.0, 127.8)
- moved C11 16.4 mm to (205.8, 106.0), turned to 90 degrees
- moved C37 15.9 mm to (205.8, 97.8), turned to 90 degrees
- moved J3 3.36 mm to (208.0, 88.2), turned to 90 degrees
- moved H1 2.35 mm to (151.0, 129.8)
- moved J6 2.02 mm to (194.2, 61.0)
- moved C1 1.93 mm to (163.5, 62.4)
Connections:
- J3 pad 1: Load1 -> Load2
- J3 pad 2: Load2 -> Load1
Routing:
- net Net-(C43-Pad1): track 15.6 -> 146.7 mm, vias 0 -> 1
- net Input: track 33.4 -> 153.5 mm
- net Load2: track 136.7 -> 132.5 mm
- net Load1: track 131.2 -> 130.3 mm
Other:
- board size 138 x 87.2 mm -> 140 x 90 mm
- board text added: "SIGNAL IN"
- board text added: "TO LOAD"
